Commit message: 新规格重建：果串 1.4-1.7 m、垄距 2.2-3.0 m 不等、加塑料大棚，机械臂换 CR10
用户给的新尺寸让原来的几何关系整个不成立，所以这次动到了机器人本体。

**为什么必须换臂。** 果串挂在 1.40-1.70 m，垄距 2.2-3.0 m，站在行间中线时到
果串的直线距离是 1.28-1.78 m，而 CR5 的包络只有约 0.95 m（0.9 m 臂展 + 95 mm
刀口）。就算贴着藤开也够不到。CR10 臂展 1.3 m，配合"贴藤行驶"把最远的果串拉回
1.23 m，不用抬高立柱、也就不用抬高重心。

**行驶车道从行间中线改成贴藤 0.80 m。** 垄距不等意味着"行间中线"到藤的距离
不是定值（1.1-1.5 m 浮动），没法作为站位基准。新增 make_models.lane_x(r)，
按固定站距 LANE_STANDOFF 贴着要采的那一垄走；aisle_x() 保留但只用于撒土块和
净空检查。drive.py 的参数相应从 _aisle 改成 _row。

场景改动：
- 垄距按种子随机（本次 2.23 / 2.72 / 2.55 m），row_x() 改为累加间距而不是乘
  固定行距，代码里不再存在"行距"这个常量。
- 每垄的结果铁丝高度独立随机（1.58-1.77 m），配合果梗长度随机，果串抓取高度
  落在 1.433-1.690 m，正好覆盖要求的 1.4-1.7 m 区间。
- 新增单体大跨拱棚 polytunnel：12.7 m 跨、脊高 5.0 m、钢管拱架每 3 m 一榀、
  五道檩条、覆膜。落地腿只在两侧最外缘，行间没有任何立柱——这是选单体大跨而
  不是连栋的原因，底盘可以走任意车道而不用绕柱子。膜只做 visual 且不投影：
  给 300 平米薄膜加碰撞体没有意义（臂最高约 2.2 m，脊在 5 m），而会投影的膜
  在 Gazebo 渲染里会把整块地压成灰的。
- 固定机位重新取景。原来那台在角落，机器人开头被裁掉一半；现在站在 row 0 车道
  外侧横向看过去，整段行程都在画面里。

CR10 换装：从 dobot_description/urdf/cr10_robot.urdf 取运动学和惯量（大臂
607 mm、小臂 568 mm，CR5 是 427/357），关节限位同样收到 ±π——厂商给的 ±6.28
会让 6 维搜索空间大约 4000 倍，RRTConnect 必超时。收拢位姿用 stow_check.py
在仿真里重测：0, -0.90, 2.40, -3.0708, -1.5708, 0，横向 0.565 m。旧的 0.45 m
横向预算是按 1.6 m 行距定的，CR10 折起来 0.565 m 会被全部否掉，已按"贴藤
0.80 m 行驶"重新推导为 0.62 m。

MoveIt 组名从 cr5_arm 改成中性的 arm：组名写在 6 个配置文件和 5 个脚本里，
带型号的名字每换一次型号就要全量追一遍，而这种陈旧耦合已经害 pick_grape.py
崩过一次。gen_srdf.py 的 stow 位姿也从 __J1__ 占位符改成命令行参数,
免得哪天真的提交一份写着 __J1__ 的 SRDF。

已验证：URDF 解析通过运动链完整；预检 39 串场景 64 个碰撞体、12 个筐位姿全部
通过碰撞感知 IK；底盘开到正对第一串车道误差 2 mm；该串的接近/抓取/退刀三个
位姿全部可解，距离 1.08-1.14 m。整行采摘尚未跑。

Co-Authored-By: NaYangyeee <93969364+NaYangyeee@users.noreply.github.com>

File: src/grape_harvest/urdf/cr10_grape.xacro (robot description, xacro)
@@ -1,6 +1,6 @@
 <?xml version="1.0"?>
-<!-- Vineyard harvesting robot: skid-steer field platform + Dobot CR5 + a
+<!-- Vineyard harvesting robot: skid-steer field platform + Dobot CR10 + a
      shear-type cutter, plus the sensors a VINS-Mono style estimator needs.
-     Arm kinematics/inertials come from dobot_gazebo/urdf/cr5_robot.xacro
+     Arm kinematics/inertials come from dobot_description/urdf/cr10_robot.urdf
      (Dobot-Arm/TCP-IP-ROS-6AXis). Differences from the vendor file:
        * <kinematic>true</kinematic> removed  -> links are real dynamic bodies
@@ -12,10 +12,15 @@
        base_footprint  ground contact point, what odometry reports
        base_link       chassis centre
-       arm_base_link   CR5 base flange, 0.75 m above the ground
-     The arm base is deliberately kept at 0.75 m, the same height the fixed
-     pedestal put it at, so the reach geometry against a 1.22 m fruiting wire
-     is unchanged. -->
-<robot name="cr5_robot" xmlns:xacro="http://ros.org/wiki/xacro">
-  <xacro:property name="mesh" value="package://dobot_description/meshes/cr5"/>
+       arm_base_link   CR10 base flange, 0.75 m above the ground
+     Why a CR10 and not the CR5 this started with: the block is planted with
+     the fruit at 1.40-1.70 m and the rows 2.2-3.0 m apart. Even hugging a row
+     at 0.80 m the straight-line distance to the highest fruit is 1.23 m, well
+     past the CR5's 0.9 m. The CR10 reaches 1.3 m, which closes the geometry
+     without raising the column and lifting the centre of gravity. Its joint
+     limits are clamped to +/-pi here for the same reason the CR5's were: the
+     vendor's +/-6.28 makes the 6-D search space about 4000x larger and
+     RRTConnect times out. -->
+<robot name="cr10_robot" xmlns:xacro="http://ros.org/wiki/xacro">
+  <xacro:property name="mesh" value="package://dobot_description/meshes/cr10"/>
   <!-- ===================== platform geometry ===================== -->
   <xacro:property name="wheel_r"    value="0.160"/>   <!-- 320 mm lug tyre -->
@@ -248,11 +253,11 @@
   <link name="arm_base_link">
     <inertial>
-      <origin xyz="-8.0961E-06 0.0019103 0.028995" rpy="0 0 0"/>
-      <mass value="0.90882"/>
-      <inertia ixx="0.0014545" ixy="4.2968E-08" ixz="-1.8199E-07"
-               iyy="0.001345"  iyz="-6.243E-06" izz="0.002155"/>
-    </inertial>
-    <visual><geometry><mesh filename="${mesh}/base_link.dae"/></geometry><material name="dobot_dark"/></visual>
-    <collision><geometry><mesh filename="${mesh}/base_link.dae"/></geometry></collision>
+      <origin xyz="-0.0017435 -4.7141E-06 0.032774" rpy="0 0 0"/>
+      <mass value="1.8265"/>
+      <inertia ixx="0.0041731" ixy="5.9354E-07" ixz="2.52E-05"
+               iyy="0.0043128"  iyz="-5.4503E-07" izz="0.0067702"/>
+    </inertial>
+    <visual><geometry><mesh filename="${mesh}/base_link.STL"/></geometry><material name="dobot_dark"/></visual>
+    <collision><geometry><mesh filename="${mesh}/base_link.STL"/></geometry></collision>
   </link>
   <joint name="arm_mount_joint" type="fixed">
@@ -260,31 +265,20 @@
     <parent link="arm_column"/><child link="arm_base_link"/>
   </joint>
-  <!-- ===================== CR5 arm ===================== -->
-  <link name="Link1">
-    <inertial>
-      <origin xyz="-8.7268E-07 -0.0032576 -0.0076748"/>
-      <mass value="1.6123"/>
-      <inertia ixx="0.0029122" ixy="5.7387E-09" ixz="1.9945E-08"
-               iyy="0.0028191" iyz="0.00044094" izz="0.0032836"/>
-    </inertial>
-    <visual><geometry><mesh filename="${mesh}/Link1.dae"/></geometry><material name="dobot_white"/></visual>
-    <collision><geometry><mesh filename="${mesh}/Link1.dae"/></geometry></collision>
-  </link>
   <joint name="joint1" type="revolute">
-    <origin xyz="0 0 0.147" rpy="0 0 0"/>
+    <origin xyz="0 0 0.1765" rpy="0 0 0"/>
     <parent link="arm_base_link"/><child link="Link1"/>
     <axis xyz="0 0 1"/>
-    <limit lower="-3.1416" upper="3.1416" effort="300" velocity="3.14"/>
-    <dynamics damping="2.0" friction="1.0"/>
-  </joint>
-  <link name="Link2">
-    <inertial>
-      <origin xyz="-0.21351 -1.3842E-06 0.14252"/>
-      <mass value="5.5186"/>
-      <inertia ixx="0.0085919" ixy="7.5552E-07" ixz="-7.8922E-07"
-               iyy="0.027553"  iyz="1.4629E-07" izz="0.028294"/>
-    </inertial>
-    <visual><geometry><mesh filename="${mesh}/Link2.dae"/></geometry><material name="dobot_white"/></visual>
-    <collision><geometry><mesh filename="${mesh}/Link2.dae"/></geometry></collision>
+    <limit lower="-3.1416" upper="3.1416" effort="500" velocity="3.14"/>
+    <dynamics damping="1.0" friction="0.5"/>
+  </joint>
+  <link name="Link1">
+    <inertial>
+      <origin xyz="-1.6635E-06 -0.010819 0.0028389" rpy="0 0 0"/>
+      <mass value="4.1649"/>
+      <inertia ixx="0.020714" ixy="-1.9343E-07" ixz="1.6036E-07"
+               iyy="0.018824"  iyz="-9.6731E-05" izz="0.014575"/>
+    </inertial>
+    <visual><geometry><mesh filename="${mesh}/Link1.STL"/></geometry><material name="dobot_white"/></visual>
+    <collision><geometry><mesh filename="${mesh}/Link1.STL"/></geometry></collision>
   </link>
   <joint name="joint2" type="revolute">
@@ -292,75 +286,85 @@
     <parent link="Link1"/><child link="Link2"/>
     <axis xyz="0 0 1"/>
-    <limit lower="-3.1416" upper="3.1416" effort="300" velocity="3.14"/>
-    <dynamics damping="2.0" friction="1.0"/>
-  </joint>
-  <link name="Link3">
-    <inertial>
-      <origin xyz="-0.15231 -1.4079E-07 0.022693"/>
-      <mass value="2.8536"/>
-      <inertia ixx="0.0032608" ixy="-3.2147E-10" ixz="0.00012363"
-               iyy="0.0092967" iyz="2.9478E-10"  izz="0.0095552"/>
-    </inertial>
-    <visual><geometry><mesh filename="${mesh}/Link3.dae"/></geometry><material name="dobot_white"/></visual>
-    <collision><geometry><mesh filename="${mesh}/Link3.dae"/></geometry></collision>
+    <limit lower="-3.1416" upper="3.1416" effort="500" velocity="3.14"/>
+    <dynamics damping="1.0" friction="0.5"/>
+  </joint>
+  <link name="Link2">
+    <inertial>
+      <origin xyz="-0.24631 3.5816E-07 0.19515" rpy="0 0 0"/>
+      <mass value="11.314"/>
+      <inertia ixx="0.033616" ixy="-8.2998E-07" ixz="-0.0033352"
+               iyy="0.30683"  iyz="-6.6457E-08" izz="0.29972"/>
+    </inertial>
+    <visual><geometry><mesh filename="${mesh}/Link2.STL"/></geometry><material name="dobot_white"/></visual>
+    <collision><geometry><mesh filename="${mesh}/Link2.STL"/></geometry></collision>
   </link>
   <joint name="joint3" type="revolute">
-    <origin xyz="-0.427 0 0"/>
+    <origin xyz="-0.607 0 0" rpy="0 0 0"/>
     <parent link="Link2"/><child link="Link3"/>
     <axis xyz="0 0 1"/>
-    <limit lower="-2.79" upper="2.79" effort="300" velocity="3.14"/>
-    <dynamics damping="2.0" friction="1.0"/>
-  </joint>
-  <link name="Link4">
-    <inertial>
-      <origin xyz="-3.2386E-07 -0.002077 -0.0015548"/>
-      <mass value="0.67058"/>
-      <inertia ixx="0.00066939" ixy="4.1975E-10" ixz="-1.0734E-08"
-               iyy="0.00065424" iyz="0.00011081" izz="0.00065365"/>
-    </inertial>
-    <visual><geometry><mesh filename="${mesh}/Link4.dae"/></geometry><material name="dobot_white"/></visual>
-    <collision><geometry><mesh filename="${mesh}/Link4.dae"/></geometry></collision>
+    <limit lower="-2.793" upper="2.793" effort="500" velocity="3.14"/>
+    <dynamics damping="1.0" friction="0.5"/>
+  </joint>
+  <link name="Link3">
+    <inertial>
+      <origin xyz="-0.2708559 2.5144691E-07 0.0622960" rpy="0 0 0"/>
+      <mass value="4.8919119"/>
+      <inertia ixx="0.0071572" ixy="-5.6201741E-07" ixz="-0.0025774807"
+               iyy="0.2396734"  iyz="9.2622830E-08" izz="0.2383692"/>
+    </inertial>
+    <visual><geometry><mesh filename="${mesh}/Link3.STL"/></geometry><material name="dobot_white"/></visual>
+    <collision><geometry><mesh filename="${mesh}/Link3.STL"/></geometry></collision>
   </link>
   <joint name="joint4" type="revolute">
-    <origin xyz="-0.357 0 0.141" rpy="0 0 -1.5708"/>
+    <origin xyz="-0.568 0 0.191" rpy="0 0 -1.5708"/>
     <parent link="Link3"/><child link="Link4"/>
     <axis xyz="0 0 1"/>
-    <limit lower="-3.1416" upper="3.1416" effort="300" velocity="3.14"/>
+    <limit lower="-3.1416" upper="3.1416" effort="500" velocity="3.14"/>
     <dynamics damping="1.0" friction="0.5"/>
   </joint>
-  <link name="Link5">
-    <inertial>
-      <origin xyz="-3.7738E-07 -0.0045777 -0.0012971"/>
-      <mass value="0.7269"/>
-      <inertia ixx="0.00073069" ixy="-5.7806E-09" ixz="6.7132E-09"
-               iyy="0.00071195" iyz="-0.00011926" izz="0.00071391"/>
-    </inertial>
-    <visual><geometry><mesh filename="${mesh}/Link5.dae"/></geometry><material name="dobot_white"/></visual>
-    <collision><geometry><mesh filename="${mesh}/Link5.dae"/></geometry></collision>
+  <link name="Link4">
+    <inertial>
+      <origin xyz="-2.5313749E-07 0.0079872450 -0.0058907423" rpy="0 0 0"/>
+      <mass value="1.1688429"/>
+      <inertia ixx="0.0029261493" ixy="8.2044008E-09" ixz="-8.1999042E-09"
+               iyy="0.0015005300"  iyz="-5.4492522E-05" izz="0.0027327494"/>
+    </inertial>
+    <visual><geometry><mesh filename="${mesh}/Link4.STL"/></geometry><material name="dobot_white"/></visual>
+    <collision><geometry><mesh filename="${mesh}/Link4.STL"/></geometry></collision>
   </link>
   <joint name="joint5" type="revolute">
-    <origin xyz="0 -0.116 0" rpy="1.5708 0 0"/>
+    <origin xyz="0 -0.125 0" rpy="1.5708 0 0"/>
     <parent link="Link4"/><child link="Link5"/>
     <axis xyz="0 0 1"/>
-    <limit lower="-3.1416" upper="3.1416" effort="300" velocity="3.14"/>
+    <limit lower="-3.1416" upper="3.1416" effort="500" velocity="3.14"/>
     <dynamics damping="1.0" friction="0.5"/>
   </joint>
-  <link name="Link6">
-    <inertial>
-      <origin xyz="5.0777E-11 9.3774E-05 -0.019285"/>
-      <mass value="0.15789"/>
-      <inertia ixx="7.8045E-05" ixy="6.1582E-15" ixz="6.2471E-14"
-               iyy="7.9168E-05" iyz="-1.3822E-07" izz="0.00012951"/>
-    </inertial>
-    <visual><geometry><mesh filename="${mesh}/Link6.dae"/></geometry><material name="dobot_white"/></visual>
-    <collision><geometry><mesh filename="${mesh}/Link6.dae"/></geometry></collision>
+  <link name="Link5">
+    <inertial>
+      <origin xyz="5.5069946E-07 -0.0145467578 -0.0045488709" rpy="0 0 0"/>
+      <mass value="1.2230308"/>
+      <inertia ixx="0.0033790546" ixy="3.5781990E-08" ixz="-7.5182806E-09"
+               iyy="0.0014925557"  iyz="8.4191792E-05" izz="0.0032330031"/>
+    </inertial>
+    <visual><geometry><mesh filename="${mesh}/Link5.STL"/></geometry><material name="dobot_white"/></visual>
+    <collision><geometry><mesh filename="${mesh}/Link5.STL"/></geometry></collision>
   </link>
   <joint name="joint6" type="revolute">
-    <origin xyz="0 0.105 0" rpy="-1.5708 0 0"/>
+    <origin xyz="0 0.1084 0" rpy="-1.5708 0 0"/>
     <parent link="Link5"/><child link="Link6"/>
     <axis xyz="0 0 1"/>
-    <limit lower="-3.1416" upper="3.1416" effort="300" velocity="3.14"/>
+    <limit lower="-3.1416" upper="3.1416" effort="500" velocity="3.14"/>
     <dynamics damping="1.0" friction="0.5"/>
   </joint>
+  <link name="Link6">
+    <inertial>
+      <origin xyz="1.4298747E-10 2.2964069E-05 -0.0205297780" rpy="0 0 0"/>
+      <mass value="0.2054395"/>
+      <inertia ixx="0.00011011543" ixy="-8.2148788E-14" ixz="4.2861584E-14"
+               iyy="0.00011066247"  iyz="3.6887993E-08" izz="0.00020518430"/>
+    </inertial>
+    <visual><geometry><mesh filename="${mesh}/Link6.STL"/></geometry><material name="dobot_white"/></visual>
+    <collision><geometry><mesh filename="${mesh}/Link6.STL"/></geometry></collision>
+  </link>
   <!-- ============ shear-type two-finger end effector ============
        The two blades close on the peduncle (fruit stem), clamp it, and cut.
