Commit message: 末端换成激光切割头 + 接料兜 + eye-in-hand RealSense；加固定起点和地面标记
**激光用 Gazebo 原生 ray 传感器建模，不是几何体凑活。** 射线能给出光束真实的
命中点和距离：会被真正挡在中间的东西遮挡，也会报距离，所以节点分得清"对准了、
0.21 m"和"立柱挡在果梗前面"。纯粹比较两个位姿的距离会让激光穿过葡萄架去切。
传感器量程 0.60 m 比激光有效射程长，有效射程 LASER_RANGE=0.35 m 在代码里判，
这样"超出射程"和"没对上"是两种可区分的失败。射线沿 laser_link 的 +Z 发射
（ray 传感器默认扫自身 XY 平面、0 度指向 +X，所以整体俯仰 -90 度），5 条射线
张角 0.7 度，工作距离上光斑约 4 mm。

**切断 = 光束在有效射程内持续照射 LASER_DWELL(1.5 s)**，中途光束脱靶就中止。
这是"能量投递"而不是几何断言。力学后果仍然走 link_attacher：先把果串固连到
末端，再解除与铁丝的连接，果串不会自由落体。

**没有夹爪之后果串靠接料兜接住。** 兜沿工具 +X（切割姿态下朝下）悬挂，顶面和
前面（+Z）敞开，所以工具前进时果串直接滑进兜里，开火前它已经站在兜里了。
放料时没有"张开"这个动作可用，只能翻腕把兜倒过来——DUMP_PITCH=-160 度让
工具 +X 的世界 z 分量变成 +0.94，兜口朝下。

夹爪相关全部清除：URDF 的 blade link/joint/传动、SRDF 的 gripper 组和
end_effector、gazebo_controllers 和 moveit_controllers 里的 gripper_controller、
joint_limits 的 blade 项、ompl_planning 的 gripper 段、pick_grape 的 gripper()。
SRDF 现在只剩 arm 一个组。stow_check 的 ARM_LINKS 补上了激光头和料兜——
料兜挂在工具下方 0.4 m，是收拢包络里最宽的东西。

**相机分工**：前桑那台前视、视野宽、随车体刚性连接，留给 VINS-Mono；新的
eye-in-hand RealSense 装在激光头上方沿光束看，留给以后的葡萄识别。两者互不干扰。

**固定起点 + 地面标记。** VINS-Mono 没有绝对参考，在哪开机就在哪建系，所以每次
从同一个位置起跑才有可比性。出生位姿收敛成 make_models.start_pose() 单一来源
（x=1.20 y=-5.20 yaw=90 度，即 row 0 工作车道上、园区南端），并在那里画一块
1.6 m 见方的标记：十字对准 base_footprint 原点、箭头指起始航向、四角黑块让它
看起来像基准而不是一摊水。只做 visual 不做碰撞——它是油漆，给它 2 cm 的碰撞
台阶正好卡在 VIO 初始化的那一刻。

已验证：URDF 解析通过运动链完整；/cut_laser/scan 正常发布（5 射线，量程
0.02-0.60）；/ee_camera/color/image_raw 和 depth/points 正常；收拢位姿在带
料兜后仍然有效。

未解决：料兜体积大，下压段笛卡尔覆盖率掉到 36%，且一旦碰到藤架，SetPosition
驱动的关节（无限刚性、没有 PID 增益）会把整台车弹开——实测一次失败后车被推移
0.79 m。这是料兜尺寸和关节刚性叠加出来的，下一轮要一起处理。

Co-Authored-By: NaYangyeee <93969364+NaYangyeee@users.noreply.github.com>

File: src/grape_harvest/urdf/cr10_grape.xacro (robot description, xacro)
@@ -1,5 +1,5 @@
 <?xml version="1.0"?>
 <!-- Vineyard harvesting robot: skid-steer field platform + Dobot CR10 + a
-     shear-type cutter, plus the sensors a VINS-Mono style estimator needs.
+     laser cutting head, plus the sensors a VINS-Mono style estimator needs.
      Arm kinematics/inertials come from dobot_description/urdf/cr10_robot.urdf
      (Dobot-Arm/TCP-IP-ROS-6AXis). Differences from the vendor file:
@@ -8,5 +8,5 @@
        * the fixed `world` joint is gone: the robot is a free body now
        * the arm sits on a wheeled platform instead of a fixed pedestal
-       * two-finger cutter on the Link6 flange
+       * laser cutting head with a catch basket on the Link6 flange
      Frames:
        base_footprint  ground contact point, what odometry reports
@@ -45,4 +45,6 @@
   <material name="chassis_y">  <color rgba="0.72 0.55 0.10 1"/></material>
   <material name="crate_wood"> <color rgba="0.62 0.44 0.20 1"/></material>
+  <material name="laser_red">  <color rgba="0.90 0.12 0.10 1"/></material>
+  <material name="basket_grey"><color rgba="0.45 0.47 0.50 1"/></material>
   <!-- ===================== chassis ===================== -->
   <link name="base_footprint"/>
@@ -367,21 +369,30 @@
     <collision><geometry><mesh filename="${mesh}/Link6.STL"/></geometry></collision>
   </link>
-  <!-- ============ shear-type two-finger end effector ============
-       The two blades close on the peduncle (fruit stem), clamp it, and cut.
-       TCP sits at the pinch point, 95 mm ahead of the Link6 flange. -->
+  <!-- ============ laser cutting head + catch basket ============
+       No jaws: the peduncle is severed by a laser, the way laser weeders burn
+       through a stem. That removes the clamp, which is what used to hold the
+       cluster, so the head carries a basket that the bunch is already sitting
+       inside when the beam fires , it drops a few centimetres onto the floor
+       of the basket rather than to the ground.
+       Frame convention for the whole head: tool +Z is the approach axis (out
+       of the Link6 flange) and tool +X points downward once the wrist is
+       pitched for a cut, so the basket hangs along +X and its opening faces
+       +Z, i.e. the bunch slides in as the tool advances.
+       TCP stays 95 mm ahead of the flange, where the beam is focused and where
+       the cut happens, so every pose in pick_grape.py keeps its meaning. -->
   <link name="ee_base">
     <inertial>
-      <origin xyz="0 0 0.028"/>
-      <mass value="0.45"/>
-      <inertia ixx="4.0E-04" ixy="0" ixz="0" iyy="4.0E-04" iyz="0" izz="4.0E-04"/>
-    </inertial>
-    <visual>
-      <origin xyz="0 0 0.028"/>
-      <geometry><box size="0.07 0.09 0.055"/></geometry>
+      <origin xyz="0 0 0.037"/>
+      <mass value="1.20"/>
+      <inertia ixx="1.6E-03" ixy="0" ixz="0" iyy="1.6E-03" iyz="0" izz="1.6E-03"/>
+    </inertial>
+    <visual>
+      <origin xyz="0 0 0.037"/>
+      <geometry><box size="0.100 0.130 0.075"/></geometry>
       <material name="dobot_dark"/>
     </visual>
     <collision>
-      <origin xyz="0 0 0.028"/>
-      <geometry><box size="0.07 0.09 0.055"/></geometry>
+      <origin xyz="0 0 0.037"/>
+      <geometry><box size="0.100 0.130 0.075"/></geometry>
     </collision>
   </link>
@@ -390,4 +401,21 @@
     <parent link="Link6"/><child link="ee_base"/>
   </joint>
+  <!-- emitter aperture; the ray sensor is attached to this link and fires
+       along its +Z -->
+  <link name="laser_link">
+    <inertial><mass value="0.05"/>
+      <inertia ixx="1e-5" ixy="0" ixz="0" iyy="1e-5" iyz="0" izz="1e-5"/>
+    </inertial>
+    <visual>
+      <origin xyz="0 0 0.006" rpy="0 0 0"/>
+      <geometry><cylinder radius="0.011" length="0.012"/></geometry>
+      <material name="laser_red"/>
+    </visual>
+  </link>
+  <joint name="laser_joint" type="fixed">
+    <origin xyz="0 0 0.075"/>
+    <parent link="ee_base"/><child link="laser_link"/>
+  </joint>
+  <!-- beam focus / nominal cut point -->
   <link name="tcp_link">
     <inertial><mass value="1e-4"/>
@@ -399,36 +427,57 @@
     <parent link="ee_base"/><child link="tcp_link"/>
   </joint>
-  <!-- q=0 -> 12 mm gap (clamped on a peduncle), q=0.042 -> 96 mm gap -->
-  <link name="left_blade">
-    <inertial><origin xyz="0 0.003 0.030"/><mass value="0.05"/>
-      <inertia ixx="2e-5" ixy="0" ixz="0" iyy="2e-5" iyz="0" izz="2e-5"/>
-    </inertial>
-    <visual><origin xyz="0 0.003 0.030"/>
-      <geometry><box size="0.05 0.006 0.062"/></geometry><material name="steel"/></visual>
-    <collision><origin xyz="0 0.003 0.030"/>
-      <geometry><box size="0.05 0.006 0.062"/></geometry></collision>
-  </link>
-  <joint name="left_blade_joint" type="prismatic">
-    <origin xyz="0 0.006 0.055"/>
-    <parent link="ee_base"/><child link="left_blade"/>
-    <axis xyz="0 1 0"/>
-    <limit lower="0.0" upper="0.042" effort="100" velocity="0.5"/>
-    <dynamics damping="5.0" friction="1.0"/>
-  </joint>
-  <link name="right_blade">
-    <inertial><origin xyz="0 -0.003 0.030"/><mass value="0.05"/>
-      <inertia ixx="2e-5" ixy="0" ixz="0" iyy="2e-5" iyz="0" izz="2e-5"/>
-    </inertial>
-    <visual><origin xyz="0 -0.003 0.030"/>
-      <geometry><box size="0.05 0.006 0.062"/></geometry><material name="steel"/></visual>
-    <collision><origin xyz="0 -0.003 0.030"/>
-      <geometry><box size="0.05 0.006 0.062"/></geometry></collision>
-  </link>
-  <joint name="right_blade_joint" type="prismatic">
-    <origin xyz="0 -0.006 0.055"/>
-    <parent link="ee_base"/><child link="right_blade"/>
-    <axis xyz="0 -1 0"/>
-    <limit lower="0.0" upper="0.042" effort="100" velocity="0.5"/>
-    <dynamics damping="5.0" friction="1.0"/>
+  <!-- eye-in-hand RealSense, above the emitter and looking down the beam.
+       Kept separate from the mast camera on purpose: this one moves with the
+       wrist, which is what fruit detection wants and what VIO does not. -->
+  <link name="ee_camera_link">
+    <inertial><mass value="0.08"/>
+      <inertia ixx="4e-5" ixy="0" ixz="0" iyy="4e-5" iyz="0" izz="4e-5"/>
+    </inertial>
+    <visual>
+      <geometry><box size="0.025 0.090 0.025"/></geometry>
+      <material name="dobot_dark"/>
+    </visual>
+    <collision>
+      <geometry><box size="0.025 0.090 0.025"/></geometry>
+    </collision>
+  </link>
+  <joint name="ee_camera_joint" type="fixed">
+    <origin xyz="-0.058 0 0.050"/>
+    <parent link="ee_base"/><child link="ee_camera_link"/>
+  </joint>
+  <link name="ee_camera_optical_frame"/>
+  <joint name="ee_camera_optical_joint" type="fixed">
+    <origin rpy="-1.5708 0 -1.5708"/>
+    <parent link="ee_camera_link"/><child link="ee_camera_optical_frame"/>
+  </joint>
+  <!-- Catch basket. Open at the top (-X) and at the front (+Z) so the tool can
+       be slid over a hanging bunch; the bunch is then standing in the basket
+       before the beam is fired. Released over the crate by pitching the wrist
+       forward so it slides out of the open front. -->
+  <xacro:macro name="basket_slab" params="x y z sx sy sz">
+    <visual>
+      <origin xyz="${x} ${y} ${z}"/>
+      <geometry><box size="${sx} ${sy} ${sz}"/></geometry>
+      <material name="basket_grey"/>
+    </visual>
+    <collision>
+      <origin xyz="${x} ${y} ${z}"/>
+      <geometry><box size="${sx} ${sy} ${sz}"/></geometry>
+    </collision>
+  </xacro:macro>
+  <link name="catch_basket">
+    <inertial>
+      <origin xyz="0.28 0 0.09"/>
+      <mass value="0.60"/>
+      <inertia ixx="6E-03" ixy="0" ixz="0" iyy="6E-03" iyz="0" izz="6E-03"/>
+    </inertial>
+    <xacro:basket_slab x="0.410" y="0"      z="0.090" sx="0.020" sy="0.240" sz="0.240"/>
+    <xacro:basket_slab x="0.275" y="0"      z="-0.030" sx="0.270" sy="0.240" sz="0.020"/>
+    <xacro:basket_slab x="0.275" y="0.120"  z="0.090" sx="0.270" sy="0.020" sz="0.240"/>
+    <xacro:basket_slab x="0.275" y="-0.120" z="0.090" sx="0.270" sy="0.020" sz="0.240"/>
+  </link>
+  <joint name="basket_joint" type="fixed">
+    <origin xyz="0 0 0"/>
+    <parent link="ee_base"/><child link="catch_basket"/>
   </joint>
   <!-- ============ ros_control transmissions (arm only) ============
@@ -454,6 +503,4 @@
   <xacro:pos_trans jname="joint5"/>
   <xacro:pos_trans jname="joint6"/>
-  <xacro:pos_trans jname="left_blade_joint"/>
-  <xacro:pos_trans jname="right_blade_joint"/>
   <!-- ===================== gazebo ===================== -->
   <gazebo>
@@ -593,12 +640,74 @@
   <xacro:tyre_surface name="wheel_rl"/>
   <xacro:tyre_surface name="wheel_rr"/>
-  <!-- high friction on the blades so the clamped peduncle does not slip -->
-  <gazebo reference="left_blade">
-    <material>Gazebo/Grey</material><mu1>2.0</mu1><mu2>2.0</mu2>
+  <gazebo reference="catch_basket">
+    <material>Gazebo/Grey</material><mu1>0.9</mu1><mu2>0.9</mu2>
     <kp>1e6</kp><kd>100</kd>
   </gazebo>
-  <gazebo reference="right_blade">
-    <material>Gazebo/Grey</material><mu1>2.0</mu1><mu2>2.0</mu2>
-    <kp>1e6</kp><kd>100</kd>
+  <gazebo reference="laser_link"><material>Gazebo/RedGlow</material></gazebo>
+  <gazebo reference="ee_camera_link"><material>Gazebo/DarkGrey</material></gazebo>
+  <!-- ============ the cutting beam ============
+       Modelled as a Gazebo ray sensor rather than a bare geometric test. The
+       ray gives the real hit point along the beam: it is occluded by whatever
+       is actually in the way, and it reports range, so the node can tell "on
+       target at 0.21 m" from "the post is in front of the stem". A pure
+       distance check between two poses would happily cut through a trellis.
+       The sensor reaches further than the laser is useful for; the effective
+       cutting range is enforced in pick_grape.py (LASER_RANGE), so the node can
+       distinguish out-of-range from off-target.
+       A ray sensor scans its own XY plane with angle 0 along +X, so it is
+       pitched -90 deg to fire along the link's +Z, which is the approach axis.
+       Five samples across 0.7 deg give a narrow beam, about 4 mm across at the
+       working distance, instead of a single ray that can slip past a stem. -->
+  <gazebo reference="laser_link">
+    <sensor name="cut_laser" type="ray">
+      <pose>0 0 0 0 -1.5708 0</pose>
+      <always_on>true</always_on>
+      <update_rate>20.0</update_rate>
+      <visualize>true</visualize>
+      <ray>
+        <scan>
+          <horizontal>
+            <samples>5</samples>
+            <resolution>1</resolution>
+            <min_angle>-0.006</min_angle>
+            <max_angle>0.006</max_angle>
+          </horizontal>
+        </scan>
+        <range>
+          <min>0.02</min>
+          <max>0.60</max>
+          <resolution>0.002</resolution>
+        </range>
+      </ray>
+      <plugin name="cut_laser_plugin" filename="libgazebo_ros_laser.so">
+        <topicName>cut_laser/scan</topicName>
+        <frameName>laser_link</frameName>
+      </plugin>
+    </sensor>
+  </gazebo>
+  <!-- eye-in-hand RealSense: for fruit detection later, not for VIO -->
+  <gazebo reference="ee_camera_link">
+    <sensor name="ee_rgbd" type="depth">
+      <always_on>true</always_on>
+      <update_rate>15.0</update_rate>
+      <camera>
+        <horizontal_fov>1.20</horizontal_fov>
+        <image><width>640</width><height>480</height><format>R8G8B8</format></image>
+        <clip><near>0.08</near><far>4.0</far></clip>
+      </camera>
+      <plugin name="ee_rgbd_plugin" filename="libgazebo_ros_openni_kinect.so">
+        <baseline>0.05</baseline>
+        <updateRate>15.0</updateRate>
+        <cameraName>ee_camera</cameraName>
+        <imageTopicName>color/image_raw</imageTopicName>
+        <cameraInfoTopicName>color/camera_info</cameraInfoTopicName>
+        <depthImageTopicName>depth/image_raw</depthImageTopicName>
+        <depthImageCameraInfoTopicName>depth/camera_info</depthImageCameraInfoTopicName>
+        <pointCloudTopicName>depth/points</pointCloudTopicName>
+        <frameName>ee_camera_optical_frame</frameName>
+        <pointCloudCutoff>0.10</pointCloudCutoff>
+        <pointCloudCutoffMax>4.0</pointCloudCutoffMax>
+      </plugin>
+    </sensor>
   </gazebo>
 </robot>

Commit message: 接料兜改成开底围栏；加底盘遥控和一键演示 launch
**接料兜是卡住机械臂的元凶，改成开底围栏。** 原来那个闭底兜挂在工具下方 0.41 m，
而臂基座 0.75 m 要够 1.55 m 的果串时是向上伸的，兜正好扫过前臂自己的空间：
抓取位姿的碰撞感知 IK 直接无解，下压段笛卡尔覆盖率掉到 36%，偶尔挤过去一次
接触就把整台车弹开 0.79 m（关节是 SetPosition 驱动的，接触等效无限刚性）。

闭底兜也没法做小：最长的果串挂在切点下方 0.47 m，兜底要躲开它只会更深。所以
改成三面围栏——围住果串稳住它，前面敞开让工具滑进去，**底部敞开所以永远不会
去顶果串**。真正托住果串的仍是 attacher 关节，这一点是诚实的：激光切不住任何
东西，总得有东西托着，围栏是这件事的机械解释而不是机构本身。开底还带来一个
好处：放料不用再翻腕倒兜，DUMP_PITCH 和它带来的 IK 风险一起去掉了。
改完下压段覆盖率从 36% 回到 **100%**。

**底盘遥控 teleop_base.py：只有前进后退，没有转向。** 臂从离垄 0.80 m 的车道上
作业，全部余量都花在这个站距上，手动转向跑偏只会把果串推出可达范围。键盘没有
抬键事件，所以指令做成 HOLD 秒后自动过期的"油门"手感。

**pick_grape.py 新增 --teleop 模式**：人开车，臂自己判断什么时候有活。车一动就
收臂，停稳 1 秒后扫一遍可达的果串，有就去切。分工是刻意的：贴多近、什么时候停
是人有直觉的部分，怎么把激光头送到果梗上不是。

**一键演示 launch/teleop_demo.launch**：Gazebo + RViz + 遥控终端 + 自动臂。
遥控要单独开一个 xterm——roslaunch 起的节点继承控制台的 stdout 但不继承 stdin，
当普通节点跑的键盘读取永远收不到按键。已验证 gzserver/gzclient/rviz/xterm/
move_group 全部起得来，/cmd_vel 能驱动底盘（5 秒走 0.345 m）。

顺带：团队提供的 CR10URDF（SolidWorks 导出）运动学参数与本仓库已有的逐项一致
（joint1 0.1765 / joint3 -0.607 / joint4 -0.568,0.191 / joint5 -0.125 /
joint6 0.1084），等于独立验证。差别只在它把所有限位写成 ±3.14，而厂商包给
joint3 是 ±2.793，保留后者。

**未解决，且已定位到具体现象：轨迹报成功但机械臂没到位。** 激光对准失败的根因
不是激光本身：开火时实测末端离指令位姿 0.54 m（末端在 [1.572,-3.734,1.882]，
指令 [2.00,-3.726,1.550]），而 compute_cartesian_path 报 100% 覆盖、execute()
报成功。把目标容差从 0.12 收到 0.01 rad、并把 allowed_start_tolerance 从 0
恢复到 0.05 之后，误差反而涨到 1.03 m、臂干脆不离开收拢姿态了——说明故障在容差
之上游，收紧容差只改变它错多远。两处配置已回退并把这个发现写在注释里。
下一轮嫌疑：world_tf.py 发的 world->odom 是否滞后或错误（MoveIt 在 world 系里
规划，这个变换错了指令位姿就落在错的地方）。

Co-Authored-By: NaYangyeee <93969364+NaYangyeee@users.noreply.github.com>

File: src/grape_harvest/urdf/cr10_grape.xacro (robot description, xacro)
@@ -451,9 +451,17 @@
     <parent link="ee_camera_link"/><child link="ee_camera_optical_frame"/>
   </joint>
-  <!-- Catch basket. Open at the top (-X) and at the front (+Z) so the tool can
-       be slid over a hanging bunch; the bunch is then standing in the basket
-       before the beam is fired. Released over the crate by pitching the wrist
-       forward so it slides out of the open front. -->
-  <xacro:macro name="basket_slab" params="x y z sx sy sz">
+  <!-- Catch collar. Three walls that surround the cluster and steady it while
+       the beam works, open at the front (+Z) so the tool slides over a hanging
+       bunch and open at the bottom so it never pushes the fruit.
+       It is deliberately NOT a closed basket. The longest bunch hangs 0.47 m
+       below the cut, so a basket with a floor under it would reach further down
+       than the forearm can tolerate: an earlier 0.41 m version made
+       collision-free IK fail at the grasp pose outright, and the contacts it
+       did produce threw the platform sideways, because SetPosition-driven
+       joints make any contact effectively rigid.
+       What actually retains the cut bunch is the attacher joint, established
+       before the cordon joint is released. A laser cannot hold anything, so
+       something has to; the collar is the mechanical account of it. -->
+  <xacro:macro name="collar_slab" params="x y z sx sy sz">
     <visual>
       <origin xyz="${x} ${y} ${z}"/>
@@ -468,12 +476,11 @@
   <link name="catch_basket">
     <inertial>
-      <origin xyz="0.28 0 0.09"/>
-      <mass value="0.60"/>
-      <inertia ixx="6E-03" ixy="0" ixz="0" iyy="6E-03" iyz="0" izz="6E-03"/>
-    </inertial>
-    <xacro:basket_slab x="0.410" y="0"      z="0.090" sx="0.020" sy="0.240" sz="0.240"/>
-    <xacro:basket_slab x="0.275" y="0"      z="-0.030" sx="0.270" sy="0.240" sz="0.020"/>
-    <xacro:basket_slab x="0.275" y="0.120"  z="0.090" sx="0.270" sy="0.020" sz="0.240"/>
-    <xacro:basket_slab x="0.275" y="-0.120" z="0.090" sx="0.270" sy="0.020" sz="0.240"/>
+      <origin xyz="0.15 0 0.09"/>
+      <mass value="0.35"/>
+      <inertia ixx="2E-03" ixy="0" ixz="0" iyy="2E-03" iyz="0" izz="2E-03"/>
+    </inertial>
+    <xacro:collar_slab x="0.150" y="0.100"  z="0.090" sx="0.180" sy="0.016" sz="0.200"/>
+    <xacro:collar_slab x="0.150" y="-0.100" z="0.090" sx="0.180" sy="0.016" sz="0.200"/>
+    <xacro:collar_slab x="0.150" y="0"      z="-0.002" sx="0.180" sy="0.216" sz="0.016"/>
   </link>
   <joint name="basket_joint" type="fixed">
@@ -675,5 +682,5 @@
         </scan>
         <range>
-          <min>0.02</min>
+          <min>0.004</min>
           <max>0.60</max>
           <resolution>0.002</resolution>
