Commit message: 找到根因：笛卡尔路径未做时间参数化就执行；激光改为有工作距离；底盘配重
**卡了很久的"轨迹报成功但机械臂没动"，根因是 compute_cartesian_path 返回的是
路径不是轨迹。** 它的路点不带时间戳，直接交给 execute() 会被接受、立刻返回成功，
而机械臂纹丝不动。之前每一次"cartesian coverage 100%"后面跟着"末端离指令位姿
0.54 m"都是这个。执行前先用 retime_trajectory 重新参数化之后，末端误差从
**0.54 m 降到 0.061 m**。

诊断过程值得记一笔：先怀疑 world_tf.py 发的 world->odom 有问题，实测 TF 与真值
差 0.0000 m、时间戳 0.02 s 新鲜，排除；又写了个最小复现（arm_check.py，只用
MoveGroup 走命名位姿和显式位姿），发现 MoveIt 关节与 /joint_states 完全一致、
显式位姿到位 2.9 mm——一切正常。差别只剩 compute_cartesian_path 这一条路径。
中途还试过收紧目标容差，当时"越收越糟"，因为那时轨迹根本没在执行，容差自然
无关；真因修掉之后容差才开始起作用。

**激光改成有工作距离的构型。** 原来发射口在 TCP 后方 15 mm 沿接近轴直射，两个
问题：比射线传感器最小量程还近，所以果梗根本不可见；而且末端 6-10 cm 的定位
误差全落在光束方向上——这是激光最不该敏感的方向，却因此把光束原点推到了果梗
后面。现在发射口移到头部上方（工具轴上方 120 mm、法兰面后 50 mm），斜向下前方
瞄准 TCP，工作距离 184 mm。这是激光切割头本来的做法，沿接近轴的误差只会让光斑
沿果梗滑动一点而不是脱靶。光束张角同时从 ±0.006 放宽到 ±0.04 rad（184 mm 处
光斑约 14 mm），因为末端横向误差约 12 mm，完全准直的光束需要谁也做不到的精度。

**结果：完整循环首次跑通。** 对位误差 22 mm → 光束在 0.057 m 处看到果梗 →
照射 1.5 s 切断 → 接住 → 退刀 100% → 搬运 100% → 释放入筐 → result: SUCCESS。

**底盘配重，不再一碰立柱就翻。** 原来整车 132 kg，其中 33 kg 是臂和立柱挂在
0.6-1.5 m 高处，重心 0.51 m 对半轮距 0.32 m，静态翻覆角只有 32 度。现在底盘
650 kg 且重心设在底盘中心下方 0.14 m（电池组装在车架底部，真实平台就是这么配的），
护板 40 kg，轮子各 18 kg：整车 802 kg、重心 0.250 m、翻覆角 **52 度**。
另外给车身加了显式的 kp/kd——Gazebo 默认接触刚度极大，撞固定立柱是刚性冲击，
能量一步全弹回车上；现在同样的撞击变成推挤。车身摩擦也调低，让它蹭着立柱滑过去
而不是挂住。实测三次故意撞击，最大 roll 8.4 度，没有翻车。

顺带修掉 report() 的判据错误：果串模型原点在果梗顶端，即使躺在筐底原点也有 0.92 m，
超过 0.77 m 的阈值，于是每次成功入筐都被报成 NOT IN CRATE。改为比较果实体中心。

Co-Authored-By: NaYangyeee <93969364+NaYangyeee@users.noreply.github.com>

File: src/grape_harvest/urdf/cr10_grape.xacro (robot description, xacro)
@@ -51,7 +51,14 @@
   <link name="base_link">
     <inertial>
-      <mass value="70.0"/>
-      <!-- box inertia for 1.50 x 0.56 x 0.22 -->
-      <inertia ixx="2.11" ixy="0" ixz="0" iyy="13.40" iyz="0" izz="14.95"/>
+      <!-- 650 kg of frame, battery and drive, with the centre of mass 0.14 m
+           below the chassis centre: the pack sits in the bottom of the frame,
+           which is where a field platform carries it and the only reason the
+           thing can survive being shoved by a post. Whole-vehicle centre of
+           mass lands near 0.25 m against a 0.32 m half-track. -->
+      <origin xyz="0 0 -0.14"/>
+      <mass value="650.0"/>
+      <!-- box inertia for 1.50 x 0.56 x 0.22, rounded up to stand in for
+           ballast spread through the frame rather than a uniform slab -->
+      <inertia ixx="25.0" ixy="0" ixz="0" iyy="130.0" iyz="0" izz="145.0"/>
     </inertial>
     <visual>
@@ -70,6 +77,8 @@
        sets the 0.25 m ground clearance over clods -->
   <link name="skid_plate">
-    <inertial><mass value="6.0"/>
-      <inertia ixx="0.2" ixy="0" ixz="0" iyy="1.0" iyz="0" izz="1.2"/>
+    <!-- 40 kg of steel plate. Heavy, and as low as anything on the vehicle
+         gets, so it earns its weight twice. -->
+    <inertial><mass value="40.0"/>
+      <inertia ixx="1.2" ixy="0" ixz="0" iyy="6.5" iyz="0" izz="7.5"/>
     </inertial>
     <visual>
@@ -96,6 +105,8 @@
     <link name="${name}_link">
       <inertial>
-        <mass value="4.0"/>
-        <inertia ixx="0.0304" ixy="0" ixz="0" iyy="0.0512" iyz="0" izz="0.0304"/>
+        <!-- 18 kg: tyre, rim and the hub gearbox behind it. iyy is the spin
+             axis (m r^2 / 2); the other two are the transverse cylinder term. -->
+        <mass value="18.0"/>
+        <inertia ixx="0.137" ixy="0" ixz="0" iyy="0.230" iyz="0" izz="0.137"/>
       </inertial>
       <visual>
@@ -132,5 +143,6 @@
       <parent link="base_link"/><child link="${name}_link"/>
       <axis xyz="0 1 0"/>
-      <limit effort="200" velocity="20"/>
+      <limit effort="900" velocity="20"/>
+      <dynamics damping="0.8" friction="2.0"/>
       <dynamics damping="0.2" friction="0.5"/>
     </joint>
@@ -403,16 +415,24 @@
   <!-- emitter aperture; the ray sensor is attached to this link and fires
        along its +Z -->
+  <!-- Emitter on top of the head, angled down-forward so the beam crosses the
+       TCP 0.184 m away. Firing straight along the approach axis from just
+       behind the tool put the stem inside the sensor's minimum range and threw
+       away the standoff a laser exists to have. -->
   <link name="laser_link">
-    <inertial><mass value="0.05"/>
-      <inertia ixx="1e-5" ixy="0" ixz="0" iyy="1e-5" iyz="0" izz="1e-5"/>
-    </inertial>
-    <visual>
-      <origin xyz="0 0 0.006" rpy="0 0 0"/>
-      <geometry><cylinder radius="0.011" length="0.012"/></geometry>
+    <inertial><mass value="0.15"/>
+      <inertia ixx="1e-4" ixy="0" ixz="0" iyy="1e-4" iyz="0" izz="1e-4"/>
+    </inertial>
+    <visual>
+      <origin xyz="0 0 0.020" rpy="0 0 0"/>
+      <geometry><cylinder radius="0.022" length="0.075"/></geometry>
       <material name="laser_red"/>
     </visual>
+    <collision>
+      <origin xyz="0 0 0.020" rpy="0 0 0"/>
+      <geometry><cylinder radius="0.022" length="0.075"/></geometry>
+    </collision>
   </link>
   <joint name="laser_joint" type="fixed">
-    <origin xyz="0 0 0.075"/>
+    <origin xyz="-0.120 0 -0.050" rpy="0 0.7086 0"/>
     <parent link="ee_base"/><child link="laser_link"/>
   </joint>
@@ -530,5 +550,8 @@
       <wheelDiameter>${2*wheel_r}</wheelDiameter>
       <robotBaseFrame>base_footprint</robotBaseFrame>
-      <torque>220</torque>
+      <!-- 900 N.m per wheel: 800 kg needs about 55 N.m total to pull away
+           at 0.5 m/s^2, but skid steering scrubs all four tyres sideways
+           through every turn and that is where the headroom goes -->
+      <torque>900</torque>
       <commandTopic>cmd_vel</commandTopic>
       <odometryTopic>odom</odometryTopic>
@@ -626,6 +649,23 @@
   </gazebo>
   <!-- materials + contact properties -->
-  <gazebo reference="base_link"><material>Gazebo/Yellow</material></gazebo>
-  <gazebo reference="skid_plate"><material>Gazebo/DarkGrey</material></gazebo>
+  <!-- Compliant contact on the bodywork. Gazebo's default stiffness resolves a
+       post strike in one step and hands the whole impulse back to the vehicle,
+       which is what was flipping it; kp here is a few hundred kN/m with heavy
+       damping, so the same strike becomes a shove. Low friction on purpose too:
+       the chassis should slide along a post it clips, not catch on it. -->
+  <gazebo reference="base_link">
+    <material>Gazebo/Yellow</material>
+    <mu1>0.35</mu1><mu2>0.35</mu2>
+    <kp>2e5</kp><kd>1500</kd>
+    <minDepth>0.003</minDepth>
+    <maxVel>0.5</maxVel>
+  </gazebo>
+  <gazebo reference="skid_plate">
+    <material>Gazebo/DarkGrey</material>
+    <mu1>0.4</mu1><mu2>0.4</mu2>
+    <kp>3e5</kp><kd>1500</kd>
+    <minDepth>0.003</minDepth>
+    <maxVel>0.5</maxVel>
+  </gazebo>
   <gazebo reference="arm_column"><material>Gazebo/DarkGrey</material></gazebo>
   <gazebo reference="arm_base_link"><material>Gazebo/DarkGrey</material></gazebo>
@@ -638,5 +678,7 @@
       <material>Gazebo/Black</material>
       <mu1>1.5</mu1><mu2>1.2</mu2>
-      <kp>1e6</kp><kd>50</kd>
+      <!-- 3e6 keeps an 800 kg vehicle from settling into the ground: at the old
+           1e6 the static deflection was 8 mm and the platform rode visibly low -->
+      <kp>3e6</kp><kd>300</kd>
       <minDepth>0.002</minDepth>
       <maxVel>1.0</maxVel>
@@ -664,6 +706,8 @@
        A ray sensor scans its own XY plane with angle 0 along +X, so it is
        pitched -90 deg to fire along the link's +Z, which is the approach axis.
-       Five samples across 0.7 deg give a narrow beam, about 4 mm across at the
-       working distance, instead of a single ray that can slip past a stem. -->
+       Nine samples across 4.6 deg give a spot about 14 mm across at the 184 mm
+       working distance. That is deliberately not a pencil beam: tool
+       positioning lands within about 12 mm laterally, and a perfectly
+       collimated beam would need accuracy nobody has. -->
   <gazebo reference="laser_link">
     <sensor name="cut_laser" type="ray">
@@ -675,8 +719,8 @@
         <scan>
           <horizontal>
-            <samples>5</samples>
+            <samples>9</samples>
             <resolution>1</resolution>
-            <min_angle>-0.006</min_angle>
-            <max_angle>0.006</max_angle>
+            <min_angle>-0.04</min_angle>
+            <max_angle>0.04</max_angle>
           </horizontal>
         </scan>

Commit message: 第 1 项 关节力矩控制：跑通并保留为可切换配置，主线仍用运动学关节
用户要求依次加入五项控制算法。第一项是关节层 PID，它是其余四项的基础——没有真实的
关节力学，力控、接触载荷、跟踪精度全都无从谈起。

**结果：力矩控制能用了，但还没整定到能跑采摘的程度，所以主线保持不变。**

`config/gazebo_controllers_torque.yaml` 是力矩版：传动接口改 EffortJointInterface，
控制器改 effort_controllers/JointTrajectoryController，PID 放在控制器里。臂由真实
关节力矩托住、不越限位、到达指令笛卡尔位姿约 17 mm——**这是本项目第一个诚实的跟踪
误差数字**（原来那个 2.9 mm 是刚性关节的假象，跟踪误差恒为零、没有物理意义）。
但命名位姿仍有约 0.10 rad 稳态误差、控制器报目标容差失败，采摘循环跑不起来。

主线因此恢复成位置/运动学版本，回归验证通过：末端 25.8 mm、激光在 0.057 m 命中、
切断、入筐 IN CRATE、result SUCCESS。文件里写清了怎么切换和下一步该调什么。

**排除掉的一条路（写在配置注释里，免得以后重试）：gazebo_ros_control 的 POSITION_PID
模式在这条链上发散。** 即使把增益压到 p=50（最多 50 N·m，远不足以举起 24 kg 的臂），
所有关节照样冲到限位，joint3 以 68 rad/s 穿透了 ±2.793 的限位跑到 -7.44 rad。
增益小到不可能驱动却仍然发散，说明是求解器的问题而非整定问题。

**另一条排除的路：暂停物理等控制器就位。** 改成力矩驱动后，从 spawn 到控制器启动的
约 2 秒里没有任何力矩托着臂，24 kg 的 CR10 会砸进自己的限位，MoveIt 随后因起始状态
越界而拒绝规划。想法是先暂停物理、控制器就位再解冻，但 Gazebo 暂停时**根本不发布
/clock**，于是所有 rospy 节点（包括控制器 spawner 本身）都卡在 init_node 等第一条
时钟消息，整个系统死锁。scripts/hold_until_ready.py 保留了这次尝试和结论。

诊断工具留下了 joint_probe 的思路：单帧快照分不清"自由落体"和"环发散"，要看轨迹。
是它显示出 joint1（竖直轴、无重力力矩）也跑到限位，才确定问题不在重力而在反馈。

Co-Authored-By: NaYangyeee <93969364+NaYangyeee@users.noreply.github.com>

File: src/grape_harvest/urdf/cr10_grape.xacro (robot description, xacro)
@@ -284,5 +284,5 @@
     <axis xyz="0 0 1"/>
     <limit lower="-3.1416" upper="3.1416" effort="500" velocity="3.14"/>
-    <dynamics damping="1.0" friction="0.5"/>
+    <dynamics damping="5.0" friction="1.0"/>
   </joint>
   <link name="Link1">
@@ -301,5 +301,5 @@
     <axis xyz="0 0 1"/>
     <limit lower="-3.1416" upper="3.1416" effort="500" velocity="3.14"/>
-    <dynamics damping="1.0" friction="0.5"/>
+    <dynamics damping="5.0" friction="1.0"/>
   </joint>
   <link name="Link2">
@@ -318,5 +318,5 @@
     <axis xyz="0 0 1"/>
     <limit lower="-2.793" upper="2.793" effort="500" velocity="3.14"/>
-    <dynamics damping="1.0" friction="0.5"/>
+    <dynamics damping="5.0" friction="1.0"/>
   </joint>
   <link name="Link3">
@@ -335,5 +335,5 @@
     <axis xyz="0 0 1"/>
     <limit lower="-3.1416" upper="3.1416" effort="500" velocity="3.14"/>
-    <dynamics damping="1.0" friction="0.5"/>
+    <dynamics damping="5.0" friction="1.0"/>
   </joint>
   <link name="Link4">
@@ -352,5 +352,5 @@
     <axis xyz="0 0 1"/>
     <limit lower="-3.1416" upper="3.1416" effort="500" velocity="3.14"/>
-    <dynamics damping="1.0" friction="0.5"/>
+    <dynamics damping="5.0" friction="1.0"/>
   </joint>
   <link name="Link5">
@@ -369,5 +369,5 @@
     <axis xyz="0 0 1"/>
     <limit lower="-3.1416" upper="3.1416" effort="500" velocity="3.14"/>
-    <dynamics damping="1.0" friction="0.5"/>
+    <dynamics damping="5.0" friction="1.0"/>
   </joint>
   <link name="Link6">
