Commit message: 力矩控制查出三个根因，跟踪误差 0.53 → 0.003 rad；力监护补上重力补偿
手腕 0.10 rad 的残差调了两轮增益（2.7x / 5x）都没用，反而更差。三个真正的
原因，没有一个是增益。

一、积分饱和。停在 stow 上测，三个关节都精确满足 Kp*e + i_clamp = 保持力矩
（误差 < 1 N·m）：joint3 -0.066/-31.1、joint4 -0.058/+4.4、joint6 -0.090/-0.9。
静置 30 秒 joint3 自己退回 0，joint4/joint6 四位小数纹丝不动。control_toolbox
在 antiwindup 关闭时只夹积分项的输出，累加器继续无限增长，冲过头就退不回来。
改为 antiwindup: true，i_clamp 按实测保持力矩重设（joint3 实测 31 N·m 却给了
300，手腕实测约 1 N·m 却给了 80）。

二、URDF 里没有电机转子的折算惯量。运动到 t=1.12 s 时 joint4 冲到 +12 rad/s、
joint6 冲到 -44 rad/s，方向相反，力矩双双钉死 ±500 N·m。那是腕部奇异点上的
差动模态失去惯量：joint5 过零时 joint4/joint6 两轴共线。真机靠减速器——转子
惯量按减速比平方折算，100:1 下 5e-5 的转子在输出端是 0.5 kg·m²；而 CAD 导出的
URDF 里 Link6 只有 1.1e-4 kg·m²，差三个数量级。Link4/5/6 惯量下限设
0.060/0.050/0.020，腕部阻尼 5 -> 15，六个关节加 implicitSpringDamper（ODE
默认显式积分阻尼，调高本身就发散）。结果：全程跟踪误差 0.53 -> 0.003 rad。

三、容差从台架动作取样是不够的。台架单条轨迹跟到 0.003 rad，据此收紧容差，
整垄一跑立刻爆（joint3 路径 0.229、joint4 终点 0.054）。按整周期实测重设为
path 0.35 / goal 0.05 / goal_time 5 s，积分增益翻倍（有 antiwindup 才安全）。
控制器中止次数 22 -> 3。

力监护（第 3、4 项）：阈值原本定在 25 N，理由是"末端自重 17.4 N，超过就是接触"，
从没实测过。补测完全无接触的自由运动：减静态偏置后中位 11.2 N、峰值 25.4 N。
阈值 25 N，噪声峰值 25.4 N——报的每一次碰撞都是末端自重在传感器系里转。用 TF
求出当前姿态的重力分量再减，噪声底降到 4.5 N（中位 0.1），阈值改 12 N，
并要求持续 0.20 s。抓到果串后重新拟合模型而不是重新取偏置。

这带出一个一直被掩盖的问题：力矩控制下，下降抓取段几乎每次都顶到果串
（joint3 路径误差 0.35 rad）。这个碰撞从第一版就存在，位置控制下关节被运动学
驱动，手臂直接硬推过去，日志一片干净。现在按阶段区分——下降/顺从/伺服段的
接触判为"到位，从这里开火"，其他阶段的接触仍然中止并放弃该串。

docs/01 加「三个不是增益的根因」，docs/03 加「难的不是触发策略，是让读数可信」，
两篇都带完整实测表格。主页状态表、已知限制、路线图、工程日志同步更新。
grape_pick_demo.launch 加 guard:=true。

Co-Authored-By: Claude Opus 5 <noreply@anthropic.com>

File: src/grape_harvest/urdf/cr10_grape.xacro (robot description, xacro)
@@ -340,5 +340,5 @@
     <axis xyz="0 0 1"/>
     <limit lower="-3.1416" upper="3.1416" effort="500" velocity="3.14"/>
-    <dynamics damping="5.0" friction="1.0"/>
+    <dynamics damping="15.0" friction="1.0"/>
   </joint>
   <link name="Link4">
@@ -346,6 +346,5 @@
       <origin xyz="-2.5313749E-07 0.0079872450 -0.0058907423" rpy="0 0 0"/>
       <mass value="1.1688429"/>
-      <inertia ixx="0.0029261493" ixy="8.2044008E-09" ixz="-8.1999042E-09"
-               iyy="0.0015005300"  iyz="-5.4492522E-05" izz="0.0027327494"/>
+      <inertia ixx="0.06" ixy="8.2044008E-09" ixz="-8.1999042E-09" iyy="0.06" iyz="-5.4492522E-05" izz="0.06" />
     </inertial>
     <visual><geometry><mesh filename="${mesh}/Link4.STL"/></geometry><material name="dobot_white"/></visual>
@@ -357,5 +356,5 @@
     <axis xyz="0 0 1"/>
     <limit lower="-3.1416" upper="3.1416" effort="500" velocity="3.14"/>
-    <dynamics damping="5.0" friction="1.0"/>
+    <dynamics damping="15.0" friction="1.0"/>
   </joint>
   <link name="Link5">
@@ -363,6 +362,5 @@
       <origin xyz="5.5069946E-07 -0.0145467578 -0.0045488709" rpy="0 0 0"/>
       <mass value="1.2230308"/>
-      <inertia ixx="0.0033790546" ixy="3.5781990E-08" ixz="-7.5182806E-09"
-               iyy="0.0014925557"  iyz="8.4191792E-05" izz="0.0032330031"/>
+      <inertia ixx="0.05" ixy="3.5781990E-08" ixz="-7.5182806E-09" iyy="0.05" iyz="8.4191792E-05" izz="0.05" />
     </inertial>
     <visual><geometry><mesh filename="${mesh}/Link5.STL"/></geometry><material name="dobot_white"/></visual>
@@ -374,5 +372,5 @@
     <axis xyz="0 0 1"/>
     <limit lower="-3.1416" upper="3.1416" effort="500" velocity="3.14"/>
-    <dynamics damping="5.0" friction="1.0"/>
+    <dynamics damping="15.0" friction="1.0"/>
   </joint>
   <link name="Link6">
@@ -380,6 +378,5 @@
       <origin xyz="1.4298747E-10 2.2964069E-05 -0.0205297780" rpy="0 0 0"/>
       <mass value="0.2054395"/>
-      <inertia ixx="0.00011011543" ixy="-8.2148788E-14" ixz="4.2861584E-14"
-               iyy="0.00011066247"  iyz="3.6887993E-08" izz="0.00020518430"/>
+      <inertia ixx="0.02" ixy="-8.2148788E-14" ixz="4.2861584E-14" iyy="0.02" iyz="3.6887993E-08" izz="0.02" />
     </inertial>
     <visual><geometry><mesh filename="${mesh}/Link6.STL"/></geometry><material name="dobot_white"/></visual>
@@ -742,4 +739,45 @@
     </sensor>
   </gazebo>
+  <!-- ODE applies <dynamics damping> explicitly, which puts an upper
+       bound on how much damping can be asked for before the integration
+       itself goes unstable. The implicit form folds it into the constraint
+       solver, which is what makes the raised wrist damping usable. -->
+  <xacro:macro name="implicit_damping" params="jname">
+    <gazebo reference="${jname}">
+      <implicitSpringDamper>true</implicitSpringDamper>
+    </gazebo>
+  </xacro:macro>
+  <xacro:implicit_damping jname="joint1"/>
+  <xacro:implicit_damping jname="joint2"/>
+  <xacro:implicit_damping jname="joint3"/>
+  <xacro:implicit_damping jname="joint4"/>
+  <xacro:implicit_damping jname="joint5"/>
+  <xacro:implicit_damping jname="joint6"/>
+  <!-- ============ wrist force/torque sensor ============
+       On ee_joint, so it reads everything past the flange: the head, the
+       collar, and whatever the collar is holding. That is the same place a
+       real machine puts it.
+       disableFixedJointLumping is not optional here. The URDF-to-SDF
+       conversion merges fixed joints into the parent link by default, and a
+       joint that has been merged out of existence cannot report a wrench;
+       provideFeedback then asks the solver to compute the constraint force
+       across it.
+       Note what this can and cannot tell you in this simulation: with the
+       joints driven by Joint::SetPosition (the default) the arm is infinitely
+       stiff, so a contact produces an impulse rather than a force that builds,
+       and the readings are spiky and not physically meaningful. Under
+       torque:=true they are. -->
+  <gazebo reference="ee_joint">
+    <disableFixedJointLumping>true</disableFixedJointLumping>
+    <provideFeedback>true</provideFeedback>
+  </gazebo>
+  <gazebo>
+    <plugin name="ee_ft_sensor" filename="libgazebo_ros_ft_sensor.so">
+      <updateRate>100.0</updateRate>
+      <topicName>ee_ft</topicName>
+      <jointName>ee_joint</jointName>
+      <gaussianNoise>0.02</gaussianNoise>
+    </plugin>
+  </gazebo>
   <!-- eye-in-hand RealSense: for fruit detection later, not for VIO -->
   <gazebo reference="ee_camera_link">
